File: Logger V1.kicad_pcb (KiCad board)
At the start: 2 copper layers, 38 parts, among them J1 USB_C_Receptacle_USB2.0_16P, Q1 SS8050, Q2 SS8050, SW1 B3U-1000P-B, SW2 B3U-1000P-B, U1 ESP32-WROOM-32E-N8, U2 TLV76733DRVR, U3 LOG Interface, U5 CH340K, U6 USBLC6-2P6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

Commit message: PCB Rev 1.0
Parts:
- added TP1: TestPoint, TestPoint:TestPoint_Pad_1.0x1.0mm, F.Cu at (150.3, 112.8)
- added TP2: TestPoint, TestPoint:TestPoint_Pad_1.0x1.0mm, F.Cu at (156.4, 112.8)
- added TP3: TestPoint, TestPoint:TestPoint_Pad_1.0x1.0mm, F.Cu at (154.4, 112.8)
- added TP4: TestPoint, TestPoint:TestPoint_Pad_1.0x1.0mm, F.Cu at (152.4, 112.8)
- C11, C13, C14, C3, C4, C6, C7, C8: footprint Capacitor_SMD:C_0603_1608Metric_Pad1.08x0.95mm_HandSolder -> Capacitor_SMD:C_0402_1005Metric_Pad0.74x0.62mm_HandSolder
- U3: moved to B.Cu
- moved U3 67.7 mm to (119.2, 105.8)
- moved D3 59.8 mm to (124.2, 86.9), turned to 90 degrees
- moved Q2 56.7 mm to (134.5, 102.3), turned to -90 degrees
- moved Q1 55.6 mm to (134.4, 96.3), turned to 90 degrees
- moved U6 51.2 mm to (127.8, 105.2), turned to 90 degrees
- moved U7 48.2 mm to (124.4, 90.7), turned to -90 degrees
- moved U2 43.1 mm to (131.3, 91.2), turned to 90 degrees
- moved R12 42.9 mm to (122.8, 86.6), turned to 90 degrees
- moved R13 41.5 mm to (125.4, 86.7), turned to 90 degrees
- moved R7 38.8 mm to (122.6, 96.8), turned to -90 degrees
- moved R2 37.1 mm to (121.9, 109.7), turned to 90 degrees
- moved C9 32.7 mm to (157.4, 88.0), turned to 180 degrees
- moved C8 31.2 mm to (157.6, 89.2), turned to 180 degrees
- moved EN 30.7 mm to (141.4, 86.5)
- moved D1 30.6 mm to (123.1, 103.4), turned to -90 degrees
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- renumbered SW1 to BOOT, SW2 to EN
Connections:
- R5 pad 2: +EXTR3V3 -> +VIN
- R6 pad 2: +EXTR3V3 -> +VIN
- R7 pad 1: /SPI_CS -> +VIN
- R7 pad 2: +EXTR3V3 -> /SPI_CS
- U1 pad 27: unconnected-(U1-IO16-Pad27) -> /UART_RX
- U1 pad 28: unconnected-(U1-IO17-Pad28) -> /UART_TX
- U1 pad 34: /UART_TX -> unconnected-(U1-RXD0/IO3-Pad34)
- U1 pad 35: /UART_RX -> unconnected-(U1-TXD0/IO1-Pad35)
- U7 pad V: (no net) -> GND
Routing:
- net +EXTR3V3: track 0.00 -> 65.9 mm, vias 0 -> 2
- net /UART_TX: track 0.00 -> 42.6 mm, vias 0 -> 2
- net /SPI_MISO: track 0.00 -> 42.0 mm, vias 0 -> 1
- net /SPI_CS: track 0.00 -> 39.6 mm, vias 0 -> 1
- net GND: track 0.00 -> 37.3 mm, vias 0 -> 70
- net /UART_RX: track 0.00 -> 36.6 mm, vias 0 -> 2
- net /SPI_SCK: track 0.00 -> 33.1 mm, vias 0 -> 1
- net +VBUS: track 0.00 -> 31.1 mm, vias 0 -> 4
- net /SPI_MOSI: track 0.00 -> 27.7 mm, vias 0 -> 1
- net +3V3: track 0.00 -> 26.9 mm
- net /PROG_EN: track 0.00 -> 25.5 mm
- net +VIN: track 0.00 -> 14.4 mm, vias 0 -> 3
- net /PROG_IO0: track 0.00 -> 13.1 mm
- net Net-(D1-K): track 0.00 -> 11.2 mm
- net +VBUSFTL: track 0.00 -> 10.3 mm
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- added copper zone on In2.Cu, net +VIN
- added copper zone on B.Cu, net GND
- added copper zone on In1.Cu, net GND
Other:
- board outline added: 50 x 30 mm
- copper layers 2 -> 4

Commit message: ATIC Logger Rev1.0
Parts:
- removed C14: 100nF, Capacitor_SMD:C_0402_1005Metric_Pad0.74x0.62mm_HandSolder
- added C5: 1uF, Capacitor_SMD:C_0603_1608Metric_Pad1.08x0.95mm_HandSolder, F.Cu at (126.0, 93.7)
- C12: value 1uF -> 100nF; footprint Capacitor_SMD:C_0603_1608Metric_Pad1.08x0.95mm_HandSolder -> Capacitor_SMD:C_0402_1005Metric_Pad0.74x0.62mm_HandSolder
- TP1: value TestPoint -> SDA
- TP2: value TestPoint -> SCL
- TP3: value TestPoint -> EXTR3V3
- TP4: value TestPoint -> GND
- moved C13 3.95 mm to (123.2, 93.4), turned to 180 degrees
- moved C12 2.05 mm to (126.8, 91.8), turned to 90 degrees
- moved TP1 0.05 mm to (150.3, 112.8)
- turned TP4 to 0 degrees
- turned TP3 to 0 degrees
- renumbered BOOT to BOOT1, EN to EN1
Connections:
- C12 pad 1: +VIN -> +3V3
- C13 pad 1: +3V3 -> +EXTR3V3
Routing:
- net GND: track 37.3 -> 38.5 mm, vias 70 -> 74
Other:
- board text added: "3V3"
- board text added: "BOOT"
- board text added: "EN"
- board text added: "GND"
- board text added: "SCL"
- board text added: "SDA"
